File: sha2017_draft_rev1_0_0.brd (EAGLE design)
At the start: 95 x 46 mm, 1 part

Commit message: criticial patch! mirror interface socket!
Parts:
- moved JP1 12.7 mm to (53.9, 51.7), flipped to the bottom
Changed lines of the file:
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@@
 <setting verticaltext="up"/>
 </settings>
-<grid distance="0.01" unitdist="mm" unit="mm" style="lines" multiple="1" display="yes" altdistance="0.025" altunitdist="inch" altunit="inch"/>
+<grid distance="1.27" unitdist="mm" unit="mm" style="lines" multiple="1" display="yes" altdistance="0.025" altunitdist="inch" altunit="inch"/>
 <layers>
 <layer number="1" name="Top" color="4" fill="1" visible="yes" active="yes"/>
@@
 <hole x="39.5" y="60.6" drill="3"/>
 <hole x="47.6" y="60.6" drill="3"/>
-<text x="40.670709375" y="47.970709375" size="1.016" layer="25" font="vector" ratio="16" rot="R45">SCL</text>
-<text x="43.24141875" y="47.958578125" size="1.016" layer="25" font="vector" ratio="16" rot="R45">IO2</text>
-<text x="45.84644375" y="48.11213125" size="1.016" layer="25" font="vector" ratio="16" rot="R45">IO1</text>
-<text x="48.44141875" y="48.01715625" size="1.016" layer="25" font="vector" ratio="16" rot="R45">IO0</text>
-<text x="53.3" y="47.775734375" size="1.016" layer="25" font="vector" ratio="16" rot="R45">GND</text>
-<text x="40.11213125" y="55.770709375" size="1.016" layer="25" font="vector" ratio="16" rot="R45">SDA</text>
-<text x="48.21715625" y="55.81715625" size="1.016" layer="25" font="vector" ratio="16" rot="R45">IO4</text>
-<text x="45.8" y="55.858578125" size="1.016" layer="25" font="vector" ratio="16" rot="R45">IO3</text>
-<text x="53.24141875" y="55.7" size="1.016" layer="25" font="vector" ratio="16" rot="R45">3V3</text>
-<text x="50.787865625" y="55.770709375" size="1.016" layer="25" font="vector" ratio="16" rot="R45">GND</text>
-<text x="43.1" y="55.8" size="1.016" layer="25" font="vector" ratio="16" rot="R45">LED</text>
-<text x="50.7" y="47.6" size="1.016" layer="25" font="vector" ratio="16" rot="R45">Vbat</text>
+<text x="53.370709375" y="47.970709375" size="1.016" layer="25" font="vector" ratio="16" rot="R45">SCL</text>
+<text x="50.86141875" y="47.958578125" size="1.016" layer="25" font="vector" ratio="16" rot="R45">IO2</text>
+<text x="48.38644375" y="48.11213125" size="1.016" layer="25" font="vector" ratio="16" rot="R45">IO1</text>
+<text x="45.90141875" y="48.01715625" size="1.016" layer="25" font="vector" ratio="16" rot="R45">IO0</text>
+<text x="40.6" y="47.775734375" size="1.016" layer="25" font="vector" ratio="16" rot="R45">GND</text>
+<text x="52.81213125" y="55.770709375" size="1.016" layer="25" font="vector" ratio="16" rot="R45">SDA</text>
+<text x="45.67715625" y="55.81715625" size="1.016" layer="25" font="vector" ratio="16" rot="R45">IO4</text>
+<text x="40.54141875" y="55.7" size="1.016" layer="25" font="vector" ratio="16" rot="R45">3V3</text>
+<text x="43.167865625" y="55.770709375" size="1.016" layer="25" font="vector" ratio="16" rot="R45">GND</text>
+<text x="43.08" y="47.6" size="1.016" layer="25" font="vector" ratio="16" rot="R45">Vbat</text>
 <dimension x1="4" y1="85" x2="4" y2="39" x3="-8.6" y3="62" textsize="1.778" layer="25"/>
 <dimension x1="0" y1="43" x2="95" y2="43" x3="47.5" y3="32.7" textsize="1.778" layer="25"/>
@@
 <hole x="39.51" y="60.6" drill="3"/>
 <hole x="47.61" y="60.6" drill="3"/>
-<text x="40.12213125" y="55.770709375" size="1.016" layer="25" font="vector" ratio="16" rot="R45">SDA</text>
-<text x="48.22715625" y="55.81715625" size="1.016" layer="25" font="vector" ratio="16" rot="R45">IO4</text>
-<text x="45.81" y="55.858578125" size="1.016" layer="25" font="vector" ratio="16" rot="R45">IO3</text>
-<text x="53.25141875" y="55.7" size="1.016" layer="25" font="vector" ratio="16" rot="R45">3V3</text>
-<text x="50.797865625" y="55.770709375" size="1.016" layer="25" font="vector" ratio="16" rot="R45">GND</text>
-<text x="43.11" y="55.8" size="1.016" layer="25" font="vector" ratio="16" rot="R45">LED</text>
+<text x="48.35" y="55.858578125" size="1.016" layer="25" font="vector" ratio="16" rot="R45">IO3</text>
+<text x="50.73" y="55.8" size="1.016" layer="25" font="vector" ratio="16" rot="R45">LED</text>
 </plain>
 <attributes>
@@
 </autorouter>
 <elements>
-<element name="JP1" library="SparkFun-Connectors" package="2X6" value="2X6 FEMALE" x="41.16" y="51.73" smashed="yes">
-<attribute name="PROD_ID" value="CONN-12423" x="41.16" y="51.73" size="1.778" layer="27" display="off"/>
-<attribute name="NAME" x="39.235" y="51.88" size="1.27" layer="25" ratio="10" rot="R90"/>
-<attribute name="VALUE" x="39.89" y="48.555" size="1.27" layer="27"/>
+<element name="JP1" library="SparkFun-Connectors" package="2X6" value="2X6 FEMALE" x="53.86" y="51.73" smashed="yes" rot="MR0">
+<attribute name="PROD_ID" value="CONN-12423" x="53.86" y="51.73" size="1.778" layer="28" rot="MR0" display="off"/>
+<attribute name="NAME" x="55.785" y="51.88" size="1.27" layer="26" ratio="10" rot="MR90"/>
+<attribute name="VALUE" x="55.13" y="48.555" size="1.27" layer="28" rot="MR0"/>
 </element>
 </elements>
@@
 </signal>
 <signal name="I2C_SCL">
-<wire x1="41.15" y1="51.73" x2="41.2" y2="51.73" width="0.4064" layer="1"/>
 <contactref element="JP1" pad="1"/>
-<wire x1="41.16" y1="51.73" x2="41.21" y2="51.73" width="0.4064" layer="1"/>
-<wire x1="41.16" y1="51.73" x2="41.15" y2="51.73" width="0" layer="19" extent="1-1"/>
 </signal>
 <signal name="N$440">
@@
 <signal name="WS2812_POWER">
 <contactref element="JP1" pad="9"/>
-<wire x1="51.32" y1="51.73" x2="51.37" y2="51.73" width="1.6764" layer="1"/>
 </signal>
 <signal name="WS2812_DATA_OUT">
@@
 <signal name="EXTIO-0">
 <contactref element="JP1" pad="7"/>
-<wire x1="48.78" y1="51.73" x2="48.83" y2="51.73" width="0.4064" layer="1"/>
 </signal>
 <signal name="EXTIO-3">
@@
 <signal name="EXTIO-1">
 <contactref element="JP1" pad="5"/>
-<wire x1="46.24" y1="51.73" x2="46.29" y2="51.73" width="0.4064" layer="1"/>
 </signal>
 <signal name="EXTIO-2">
 <contactref element="JP1" pad="3"/>
-<wire x1="43.7" y1="51.73" x2="43.75" y2="51.73" width="0" layer="19" extent="1-16"/>
 </signal>
 <signal name="EXTIO-4">
